Commit message: c

File: src/envs/cartpole_pbt/cartpole.urdf (robot description, URDF)
Before this commit: robot physics, 3 links, 2 joints
Links:
- link cart: geometry visual box size=0.5 0.5 0.2
- link pole: mass 0.1 -> 1.0
Joints:
- joint cart_to_pole: limit (none) -> lower=-2 upper=2 effort=1000.0 velocity=10
- joint slider_to_cart: limit lower=-15 upper=15 effort=1000.0 velocity=5 -> lower=-2 upper=2 effort=1000.0 velocity=10

Commit message: c

File: src/envs/cartpole_pbt/cartpole.urdf (robot description, URDF)
Before this commit: robot physics, 3 links, 2 joints
Links:
- link pole: geometry collision box size=0.05 0.05 1.0; visual sphere radius=0.1

Commit message: 2

File: src/envs/cartpole_pbt/cartpole.urdf (robot description, URDF)
Before this commit: robot physics, 3 links, 2 joints
Links:
- removed link pole
- added link sphere, mass 1.0; collision box size=0.05 0.05 1.0; visual sphere radius=0.1
Joints:
- removed joint cart_to_pole
- added joint swing: type continuous, parent cart, child sphere, origin xyz=0.0 0.0 0, axis 0 1 0, limit lower=-2 upper=2 effort=1000.0 velocity=10

Commit message: c

File: src/envs/cartpole_pbt/cartpole.urdf (robot description, URDF)
Before this commit: robot physics, 3 links, 2 joints
Joints:
- joint slider_to_cart: limit lower=-2 upper=2 effort=1000.0 velocity=10 -> lower=-3 upper=3 effort=1000.0 velocity=5
