Commit message: c

File: src/envs/cartpole_pbt/cartpole_balance.urdf (robot description, URDF)
Before this commit: robot physics, 4 links, 3 joints
Links:
- removed link pole_1
- removed link pole_2
- added link pole, mass 10; collision box size=0.05 0.05 1.0; visual box size=0.05 0.05 1.0
- added link weight, mass 1.0; collision box size=0.05 0.05 1.0; visual sphere radius=0.1
- link cart: geometry collision box size=0.5 0.5 0.2; visual box size=0.5 0.5 0.2
Joints:
- removed joint swing_1
- removed joint swing_2
- added joint cart_to_pole: type continuous, parent cart, child pole, origin xyz=0.0 0.0 0, axis 0 1 0
- added joint sphere_to_pole: type prismatic, parent pole, child weight, origin xyz=0.0 0.0 0.0, axis 0 0 1, limit lower=-15 upper=15 effort=1000.0 velocity=5
- joint slider_to_cart: limit lower=-3 upper=3 effort=1000.0 velocity=5 -> lower=-15 upper=15 effort=1000.0 velocity=5

File: src/envs/cartpole_pbt/hangpole_vl.urdf (robot description, URDF)
Before this commit: robot physics, 4 links, 3 joints
Links:
- removed link pole_1
- removed link pole_2
- added link sphere, mass 1.0; collision box size=0.05 0.05 1.0; visual sphere radius=0.1
Joints:
- removed joint swing_1
- removed joint swing_2
- added joint swing: type continuous, parent cart, child sphere, origin xyz=0.0 0.0 0, axis 0 1 0, limit lower=-2 upper=2 effort=1000.0 velocity=10

Commit message: c

File: src/envs/cartpole_pbt/cartpole_balance.urdf (robot description, URDF)
Before this commit: robot physics, 4 links, 3 joints
Links:
- link pole: mass 10 -> 1
